File: trunk/EI/hw/Xbee-MCP-adapter.kicad_pcb (KiCad board)
At the start: 2 copper layers, 11 parts, among them K1 POT-10K, P1 MCPboard-J3, P2 MCPboard-j4, U1 XBEE

Commit message: placa final
Routing:
- net VDD: track 77.5 -> 79.3 mm
- net /MCPboard-RTS: track 70.5 -> 71.7 mm
- net /MCPboard-CTS: track 66.5 -> 65.4 mm
Other:
- board text added: "- POT +"
- board text added: "3.3V"
- board text added: "AN0"
- board text added: "CTS"
- board text added: "DO1"
- board text added: "DO2"
- board text added: "GND"
- board text added: "RTS"
- board text added: "RXD"
- board text added: "TXD"
- board text added: "Xbee-MCP Adapter ESE - IUA - 2016"
- board text added: "~RESET"
